Commit message: everything is working

File: robot_description/urdf/robot_2.urdf.xacro (robot description, xacro)
@@ -241,5 +241,5 @@
     <origin xyz="0  0.024 0.02" rpy="0 0 0"/>
     <axis xyz="0 1 0"/>
-    <limit lower="0.0" upper="0.03" effort="20" velocity="0.1"/>
+    <limit lower="0.0" upper="0.03" effort="200" velocity="0.1"/>
     <dynamics damping="0.1" friction="0.05"/>
   </joint>
@@ -249,5 +249,5 @@
     <origin xyz="0 -0.024 0.02" rpy="0 0 0"/>
     <axis xyz="0 -1 0"/>
-    <limit lower="0.0" upper="0.03" effort="20" velocity="0.1"/>
+    <limit lower="0.0" upper="0.03" effort="200" velocity="0.1"/>
     <dynamics damping="0.1" friction="0.05"/>
     <mimic joint="finger_left_joint" multiplier="1" offset="0"/>
@@ -332,4 +332,10 @@
         <param name="max">0.03</param>
       </command_interface>
+      <state_interface name="position"><param name="initial_value">0.0</param></state_interface>
+      <state_interface name="velocity"/>
+      <state_interface name="effort"/>
+    </joint>
+    <!-- finger_right mirrors finger_left via the URDF <mimic> tag; no command interface -->
+    <joint name="finger_right_joint">
       <state_interface name="position"><param name="initial_value">0.0</param></state_interface>
       <state_interface name="velocity"/>
@@ -343,4 +349,22 @@
       <parameters>$(find robot_simulation)/config/ros2_controllers.yaml</parameters>
     </plugin>
+  </gazebo>
+  <!-- ── Gazebo: finger friction ────────────────────────────────── -->
+  <!-- urdf2sdf expects flat tags inside <gazebo reference>, NOT nested SDF -->
+  <gazebo reference="finger_left">
+    <mu1>5.0</mu1>
+    <mu2>5.0</mu2>
+    <kp>1e6</kp>
+    <kd>1.0</kd>
+    <minDepth>0.001</minDepth>
+    <maxVel>0.1</maxVel>
+  </gazebo>
+  <gazebo reference="finger_right">
+    <mu1>5.0</mu1>
+    <mu2>5.0</mu2>
+    <kp>1e6</kp>
+    <kd>1.0</kd>
+    <minDepth>0.001</minDepth>
+    <maxVel>0.1</maxVel>
   </gazebo>
   <!-- ── Gazebo: RGBD camera sensor ──────────────────────────── -->
